File: Breeze.kicad_pcb (KiCad board)
At the start: 2 copper layers, 210.6 x 114.9 mm, 102 parts, among them J1 PJ-320A, SW1 CHOCXHSPCB-1U, SW10 CHOCXHSPCB-1U, SW11 CHOCXHSPCB-1U, SW12 CHOCXHSPCB-1U, SW13 CHOCXHSPCB-1U, SW14 CHOCXHSPCB-1U, SW15 CHOCXHSPCB-1U, SW16 CHOCXHSPCB-1U, SW17 CHOCXHSPCB-1U, SW18 CHOCXHSPCB-1U, SW19 CHOCXHSPCB-1U, SW2 CHOCXHSPCB-1U, SW20 CHOCXHSPCB-1U, SW21 CHOCXHSPCB-1U, SW22 CHOCXHSPCB-1U, SW23 CHOCXHSPCB-1U, SW24 CHOCXHSPCB-1U, SW3 CHOCXHSPCB-1U, SW4 CHOCXHSPCB-1U, SW5 CHOCXHSPCB-1U, SW6 CHOCXHSPCB-1U, SW7 CHOCXHSPCB-1U, SW8 CHOCXHSPCB-1U, SW9 CHOCXHSPCB-1U

Commit message: Buncho PCB Changes
Parts:
- added G***: LOGO, RoseArt:RoseLogo, F.Cu at (129.8, 157.2)
- D1, D10, D11, D12, D13, D14, D15, D16, D17, D18, D19, D2, D20, D21, D22, D23, D24, D3, D4, D5, D6, D7, D8, D9, DALF1, DAN1, DMC1, DMC2, DMC3, DMC4, DMC5, DMC6, DRT1, DTC1, DTC2, DTC3, DTC4, DUP1: footprint Breeze:SOD-123FL -> Diode_SMD:D_SOD-123F
- moved LGO1 4.48 mm to (121.3, 156.8)
- moved DMC1 3.00 mm to (266.4, 120.8)
- moved DMC5 1.45 mm to (280.9, 120.7)
- moved RSW1 1.21 mm to (114.4, 163.1)
- moved DMC6 0.95 mm to (304.5, 120.7)
- renumbered DOWN to DOWN1, LEFT to LEFT1, RIGHT to RIGHT1, UP to UP1
Connections:
- MCU-MACRO1 pad 10: Net-(MCU-MACRO1-Pad10) -> unconnected-(MCU-MACRO1-VCC-Pad10)
- MCU-MACRO1 pad 7: Net-(MCU-MACRO1-Pad7) -> unconnected-(MCU-MACRO1-RAW-Pad7)
- MCU-MAIN1 pad 1: Net-(MCU-MAIN1-Pad1) -> unconnected-(MCU-MAIN1-TX(PD3)-Pad1)
- MCU-MAIN1 pad 13: Net-(MCU-MAIN1-Pad13) -> unconnected-(MCU-MAIN1-D10(PB6)-Pad13)
- MCU-MAIN1 pad 24: Net-(MCU-MAIN1-Pad24) -> unconnected-(MCU-MAIN1-RAW-Pad24)
Routing:
- net unconnected-(MCU-MAIN1-TX(PD3)-Pad1): track 0.00 -> 17.0 mm, vias 0 -> 1
- net Net-(MCU-MAIN1-Pad1): track 17.0 -> 0.00 mm, vias 1 -> 0
- net unconnected-(MCU-MAIN1-D10(PB6)-Pad13): track 0.00 -> 14.7 mm
- net Net-(MCU-MAIN1-Pad13): track 14.7 -> 0.00 mm
- net unconnected-(MCU-MAIN1-RAW-Pad24): track 0.00 -> 14.4 mm
- net Net-(MCU-MAIN1-Pad24): track 14.4 -> 0.00 mm
- net GND: track 408.5 -> 399.7 mm
- net ROW0: track 288.5 -> 291.8 mm
- net Net-(DMC1-A): track 44.9 -> 42.6 mm
- net ROW1: track 272.2 -> 270.0 mm
- net Net-(DMC5-A): track 41.3 -> 39.9 mm
- net Net-(DMC6-A): track 46.4 -> 45.4 mm
- net RST: track 50.2 -> 50.9 mm
- net Net-(D11-A): track 51.5 -> 50.9 mm
Other:
- board text added: "JLCJLCJLCJLC"
- board text added: "Ocean waves, open window, sunlit breeze."
- board text added: "Snap-Off for Right Hand"
- board text removed: "Snap-Off for Left Hand"
