File: Breeze.kicad_sch (KiCad schematic)
At the start: 102 parts

Commit message: Buncho PCB Changes
Parts:
- removed J1: (no value), symbol Breeze-rescue:MJ-4PP-9-Lily58-cache-Merkaba_Rev0-rescue-Breeze-rescue
- D1, D10, D11, D12, D13, D14, D15, D16, D17, D18, D19, D2, D20, D21, D22, D23, D24, D3, D4, D5, D6, D7, D8, D9, DALF1, DAN1, DMC1, DMC2, DMC3, DMC4, DMC5, DMC6, DRT1, DTC1, DTC2, DTC3, DTC4, DUP1: value (none) -> DIODE; footprint (none) -> Diode_SMD:D_SOD-123F; JLCPCB Part # (none) -> C391324
- DOWN1, LEFT1, MC1, MC2, MC3, MC4, MC5, MC6, RIGHT1, SW1, SW10, SW11, SW12, SW13, SW14, SW15, SW16, SW17, SW18, SW19, SW2, SW20, SW21, SW22, SW23, SW24, SW3, SW4, SW5, SW6, SW7, SW8, SW9, TC1, TC2, TC3, TC4, UP1: value (none) -> CHOCXHSPCB-1U; footprint (none) -> Breeze:MX_Choc_Hotswap
- H1, H16, H17, H18, H19, H2, H3, H4, H5, H6, H7, H8, H9: value (none) -> M3-HOLE; footprint (none) -> Breeze:M3-HOLE
- H10, H11, H12, H13, H14, H15: value (none) -> 2M-HOLE; footprint (none) -> Breeze:M2-HOLE
- LGO1: value (none) -> Logo; footprint (none) -> Breeze:logo
- MCU-MACRO1: value (none) -> ProMicro-Partial; footprint (none) -> Breeze:PROMICRO-PARTIAL2
- MCU-MAIN1: value (none) -> PRO-MICRO; footprint (none) -> Breeze:ProMicro
- RSW-MACRO1, RSW1: value (none) -> SW-RST; footprint (none) -> Breeze:TACT_SWITCH_TVBP06
- STABL1: value (none) -> MX-STABILIZER-2U; footprint (none) -> Breeze:Stabilizer_MX_2u
